File: tlacitko2024/tlacitko2024.kicad_sch (KiCad schematic)
At the start: 1 part, among them J1 USB_C_Receptacle_PowerOnly_6P

Commit message: 1
Parts:
- added U1: ESP32-WROOM-32, RF_Module:ESP32-WROOM-32, symbol RF_Module:ESP32-WROOM-32
Connections:
- new net: U1.1 (GND), U1.15 (GND), U1.38 (GND), U1.39 (GND)
Changed lines of the file:
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@@
 (kicad_sch (version 20230121) (generator eeschema)
   (paper "A4")
+  (symbol (lib_id "RF_Module:ESP32-WROOM-32") (at 120.65 63.5 0) (unit 1)
+    (in_bom yes) (on_board yes) (dnp no) (fields_autoplaced)
+    (property "Reference" "U1" (at 122.8441 25.4 0)
+      (effects (font (size 1.27 1.27)) (justify left))
+    )
+    (property "Value" "ESP32-WROOM-32" (at 122.8441 27.94 0)
+      (effects (font (size 1.27 1.27)) (justify left))
+    )
+    (property "Footprint" "RF_Module:ESP32-WROOM-32" (at 120.65 101.6 0)
+      (effects (font (size 1.27 1.27)) hide)
+    )
+    (property "Datasheet" "https://www.espressif.com/sites/default/files/documentation/esp32-wroom-32_datasheet_en.pdf" (at 113.03 62.23 0)
+      (effects (font (size 1.27 1.27)) hide)
+    )
+    (pin "22")
+    (pin "3")
+    (pin "27")
+    (pin "26")
+    (pin "29")
+    (pin "21")
+    (pin "10")
+    (pin "39")
+    (pin "15")
+    (pin "12")
+    (pin "1")
+    (pin "7")
+    (pin "31")
+    (pin "37")
+    (pin "25")
+    (pin "4")
+    (pin "35")
+    (pin "9")
+    (pin "17")
+    (pin "6")
+    (pin "36")
+    (pin "23")
+    (pin "38")
+    (pin "20")
+    (pin "33")
+    (pin "5")
+    (pin "19")
+    (pin "14")
+    (pin "16")
+    (pin "32")
+    (pin "2")
+    (pin "24")
+    (pin "18")
+    (pin "11")
+    (pin "13")
+    (pin "28")
+    (pin "34")
+    (pin "8")
+    (pin "30")
+    (instances
+      (project "tlacitko2024"
+        (path "/a0a40220-b244-4ec3-8b83-1977826e8278"
+          (reference "U1") (unit 1)
+        )
+      )
+    )
+  )
   (symbol (lib_id "Connector:USB_C_Receptacle_PowerOnly_6P") (at 45.72 67.31 0) (unit 1)
     (in_bom yes) (on_board yes) (dnp no) (fields_autoplaced)
