File: pd65hotplate_esp32/pd65hotplate_esp32.kicad_sch (KiCad schematic)
At the start: 16 parts, among them U1 TPS54202DDCR, U2 HUSB238_002DD, U3 ESP32-S3-WROOM-1U-N16R8, U4 STUSB4500QTR, U5 HUSB238A

Commit message: 3
Parts:
- added U6: LMR38020SDDAR, easyeda2kicad:ESOP-8_L4.9-W3.9-P1.27-LS6.0-BL-EP-1, symbol EasyEda2Kicad:LMR38020SDDAR
Connections:
- net CC1: now also U5.3 (CC1)
- net CC2: now also U5.4 (CC2)
- net DN: now also U5.2 (D-)
- net DP: now also U5.1 (D+)
- net GND: now also U5.17 (GND)
- net SCL: now also U5.10 (SCL/SNK_ISET)
- net SDA: now also U5.9 (SDA/SNK_VSET)
- net at U5.16 (VBUS): now also C3.1, R2.2, U2.1 (VIN)
Other:
- moved on the sheet: U4, U5

Commit message: obr
Connections:
- net GND: now also U6.1 (GND)
- net Vbus: now also U6.3 (VIN)
Other:
- moved on the sheet: U6

Commit message: ř
Parts:
- added C10, C7, C9: 22u, symbol Device:C
- added C4, C8: 100n, symbol Device:C
- added C5: 10u, symbol Device:C
- added C6: 220p, symbol Device:C
- added L2: 22uH 48mOhm, symbol Device:L
- added R1: 64k9, symbol Device:R
- added R3: 100k, symbol Device:R
- added R4: 23k2, symbol Device:R
- added R5: 10k, symbol Device:R
Connections:
- net 3V3: now also C10.1, C6.1, C7.1, C9.1, L2.2, R3.1, R4.1
- net GND: now also U6.9 (EP), C10.2, C4.2, C5.2, C7.2, C9.2, R1.2, R5.2
- net Vbus: now also U6.2 (EN), C4.1, C5.1
- net at U6.4 (RT/SYNC): now also R1.1
- net at U6.5 (FB): now also C6.2, R4.2, R5.1
- net at U6.6 (PG): now also R3.2
- net at U6.7 (BOOT): now also C8.1
- net at U6.8 (SW): now also C8.2, L2.1
Other:
- moved on the sheet: C1, C2, Cbst1, Cff1, D1, L1, Rfbb1, Rfbt1, U1, U6, USB1

Commit message: prac
Parts:
- removed C1: 6.8u 3.8mOhm, symbol Device:C
- removed C10, C9: 22u, symbol Device:C
- removed C2: 47uF 3mOhm, symbol Device:C
- removed C3: 105K50V, symbol Device:C
- removed C4, C8: 100n, symbol Device:C
- removed C5: 10u, symbol Device:C
- removed C6: 220p, symbol Device:C
- removed Cbst1: 100n 64mOhm, symbol Device:C
- removed Cff1: 56p, symbol Device:C
- removed L1: 5.6uH 120mOhm, symbol Device:L
- removed L2: 22uH 48mOhm, symbol Device:L
- removed R1: 64k9, symbol Device:R
- removed Rfbb1: 22k1, symbol Device:R
- removed Rfbt1: 100k, symbol Device:R
- removed U1: TPS54202DDCR, easyeda2kicad:SOT-23-6_L2.9-W1.6-P0.95-LS2.8-BL, symbol EasyEda2Kicad:TPS54202DDCR
- removed U2: HUSB238_002DD, easyeda2kicad:DFN-10_L3.0-W3.0-P0.50-BL-EP2.5, symbol EasyEda2Kicad:HUSB238_002DD
- removed U4: STUSB4500QTR, easyeda2kicad:QFN-24_L4.0-W4.0-P0.50-BL-EP2.8, symbol EasyEda2Kicad:STUSB4500QTR
- removed U6: LMR38020SDDAR, easyeda2kicad:ESOP-8_L4.9-W3.9-P1.27-LS6.0-BL-EP-1, symbol EasyEda2Kicad:LMR38020SDDAR
- added C?, Cinx1: 220n/100V, Capacitor_SMD:C_1206_3216Metric, symbol Device:C
- added Cboot1: GRM155R71A104KA01D, easyeda2kicad:C0402, symbol EasyEda2Kicad:GRM155R71A104KA01D
- added Cin1: GCM32DC72A475KE02L, easyeda2kicad:C1210, symbol EasyEda2Kicad:GCM32DC72A475KE02L
- added Cout1, Cout2, Cout3: GRM32ER61C476KE15L, easyeda2kicad:C1210, symbol EasyEda2Kicad:GRM32ER61C476KE15L
- added Cvcc1: EMK107B7105KA-T, easyeda2kicad:C0603, symbol EasyEda2Kicad:EMK107B7105KA-T
- added D3: 10-18v, symbol Device:D_Zener_Small
- added IC1: LMR36510FADDAR, SamacSys_Parts:SOIC127P600X170-9N, symbol SamacSys_Parts:LMR36510FADDAR
- added JP1: SolderJumper_3_Open, symbol Jumper:SolderJumper_3_Open
- added JP2, JP3: SolderJumper_3_Open, TestPoint:TestPoint_2Pads_Pitch2.54mm_Drill0.8mm, symbol Jumper:SolderJumper_3_Open
- added L2: SDR1105-220ML, easyeda2kicad:IND-SMD_L11.0-W10.0-2, symbol EasyEda2Kicad:SDR1105-220ML
- added Q1: PMOS, symbol Simulation_SPICE:PMOS
- added R10, R11, R12, R13, R14, R15, R16, R17, R18, R19, R20, R21, R22, R23, R24, R6: R, symbol Device:R
- added R2: 900k, Resistor_SMD:R_0603_1608Metric_Pad0.98x0.95mm_HandSolder, symbol Device:R
- added R8: ~, Resistor_SMD:R_0603_1608Metric_Pad0.98x0.95mm_HandSolder, symbol Device:R
- added R9: ~, easyeda2kicad:R0402, symbol Device:R
- added R?: 920k, Resistor_SMD:R_0603_1608Metric_Pad0.98x0.95mm_HandSolder, symbol Device:R
- added R?: 50k, easyeda2kicad:R0402, symbol Device:R
- added Renb1, Rtfb1: CRCW0402100KFKED, easyeda2kicad:R0402, symbol Device:R
- added Rent1: CRCW0402100KFKED, Resistor_SMD:R_0603_1608Metric_Pad0.98x0.95mm_HandSolder, symbol Device:R
- added Rpg1: CRCW0402100KFKED, easyeda2kicad:R0402, symbol EasyEda2Kicad:CRCW0402100KFKED
- added Rtbb1: CRCW040243K2FKED, easyeda2kicad:R0402, symbol Device:R
- added TP1: TestPoint, symbol Connector:TestPoint
- added U1: RT9068GSP, easyeda2kicad:ESOP-8_L4.9-W3.9-P1.27-LS6.0-BL-EP2.3, symbol EasyEda2Kicad:RT9068GSP
- added U3, U4: 74HC4051M/TR, Package_DIP:DIP-16_W7.62mm_SMDSocket_SmallPads, symbol EasyEda2Kicad:74HC4051M_TR
- C7: value 22u -> 22p; footprint (none) -> Capacitor_SMD:C_0805_2012Metric_Pad1.18x1.45mm_HandSolder; now not fitted
- R1: renamed from R2; footprint (none) -> Resistor_SMD:R_0603_1608Metric_Pad0.98x0.95mm_HandSolder
- R3: value 100k -> 900k; footprint (none) -> Resistor_SMD:R_0603_1608Metric_Pad0.98x0.95mm_HandSolder
- R4: value 23k2 -> 900k; footprint (none) -> Resistor_SMD:R_0603_1608Metric_Pad0.98x0.95mm_HandSolder
- R5: value 10k -> R
- renumbered U3 to U2, U5 to U6
Connections:
- net 3V3: now also Cout1.2, Cout2.2, L2.1, Rpg1.2, Rtfb1.1, U3.16 (VCC), U4.16 (VCC); no longer R3.1, R4.1
- net GND: now also U6.12 (EN_N), C?.2, Cin1.2, Cinx1.2, Cout1.1, Cout2.1, Cout3.1, Cvcc1.1, IC1.1 (PGND), IC1.9 (THERMAL), JP1.3 (B), R10.1, R11.1, R12.1, R13.2, R14.2, R15.2, R16.2, R17.1, R18.1, R19.1, R20.1, R21.2, R22.2, R23.2, R24.2, R6.1, R?.2, Renb1.2, Rtbb1.2, U1.5 (SHDN), U1.6 (GND), U1.7 (GND), U1.9 (EP), U3.7 (VEE), U3.8 (GND), U4.7 (VEE), U4.8 (GND); no longer C7.2, R5.2
- net SCL: now also JP3.1 (A); no longer U6.10 (SCL/SNK_ISET)
- net SDA: now also JP2.1 (A); no longer U6.9 (SDA/SNK_VSET)
- net Vbus: now also C?.1, Cin1.1, Cinx1.1, D3.1 (K), IC1.2 (VIN), Q1.3 (S), R8.1, Rent1.1, U1.8 (VIN); no longer R1.1
- net at R4.2: now also U6.6 (DBG_N); no longer R5.1
- net INT: now reaches U6.11 (INT_N)
- net INT: now also R5.1
- net at U6.15 (GATE): now also R9.2
- net at U6.5 (VDD): now also R3.1, R4.1, R5.2, JP1.1 (A)
- net at U6.7 (EN_HVDCP/OUT1): now also R3.2
- net at U6.8 (ADDR/ORIENT): now also R2.2
- new net: R21.1, U4.15 (A2)
- new net: JP2.2 (C), U6.9 (SDA/SNK_VSET)
- new net: JP2.3 (B), U3.3 (COMOUT/INA)
- new net: R14.1, U3.14 (A1)
- new net: Cout3.2, R1.1, R?.1, TP1.1, U1.1 (VOUT), U1.2 (SENSE)
- new net: R?.1, R?.2, U1.3 (FB)
- new net: Cboot1.1, IC1.8 (SW), L2.2
- new net: Cboot1.2, IC1.7 (BOOT)
- new net: R23.1, U4.13 (A0)
- new net: JP3.2 (C), U6.10 (SCL/SNK_ISET)
- new net: R19.2, U4.4 (A7)
- new net: IC1.3 (EN), Renb1.1, Rent1.2
- new net: IC1.4 (PG), Rpg1.1
- new net: C7.2, IC1.5 (FB), Rtbb1.1, Rtfb1.2
- new net: Cvcc1.2, IC1.6 (VCC)
- new net: R6.2, U3.1 (A4)
- new net: R16.1, U3.12 (A3)
- new net: R15.1, U3.13 (A0)
- new net: R13.1, U3.15 (A2)
- new net: R10.2, U3.2 (A6)
- new net: R11.2, U3.4 (A7)
- new net: R12.2, U3.5 (A5)
- new net: D3.2 (A), Q1.2 (G), R8.2, R9.1
- new net: R17.2, U4.1 (A4)
- new net: R22.1, U4.14 (A1)
- new net: JP1.2 (C), R2.1
- new net: R24.1, U4.12 (A3)
- new net: R20.2, U4.5 (A5)
- new net: R18.2, U4.2 (A6)
- new net: JP3.3 (B), U4.3 (COMOUT/INA)
Other:
- note added: "4.2V-65V to 3.30V @ 1A"
- note added: "Open GPIO mode 2+1(VDD) I2C 62H 2+3(GND) I2C 42H"
- note added: "R2 V 48k 24.61 49k 24.09...e96 50k 23.59 51k 23.11...e96 52k 22.65 ​ ​"
- note removed: "4.5-20V in, 3V3/800mA out"
- moved on the sheet: D1, R1, U2, U6, USB1

Commit message: add supercap backup
Parts:
- removed JP1: SolderJumper_3_Open, symbol Jumper:SolderJumper_3_Open
- removed JP2, JP3: SolderJumper_3_Open, TestPoint:TestPoint_2Pads_Pitch2.54mm_Drill0.8mm, symbol Jumper:SolderJumper_3_Open
- removed R12, R19: R, symbol Device:R
- removed U3, U4: 74HC4051M/TR, Package_DIP:DIP-16_W7.62mm_SMDSocket_SmallPads, symbol EasyEda2Kicad:74HC4051M_TR
- added C10, C2, C3: 1u, symbol Device:C
- added C11: 100n, symbol Device:C_Small
- added C5, C6, C8: 10u, symbol Device:C_Small
- added C7: 20u, symbol Device:C_Small
- added C9: DGH155Q5R5, CAPPRD350W60D825H1850, symbol SamacSys_Parts:DGH155Q5R5
- added D3: PESD4USB5U-TTSX, SamacSys_Parts:PESD4USB5UTTSX, symbol SamacSys_Parts:PESD4USB5U-TTSX
- added D4: BAT54S, Package_TO_SOT_SMD:SOT-23, symbol Diode:BAT54S
- added D5: BAT54SDW, Package_TO_SOT_SMD:SOT-363_SC-70-6, symbol Diode:BAT54SDW
- added IC2: BQ25173QWDRCRQ1, SamacSys_Parts:BQ25173QWDRCRQ1, symbol SamacSys_Parts:BQ25173QWDRCRQ1
- added IC3: TPS61299YBHR/TPS612997, BGA6C40P2X3_84X123X40, symbol SamacSys_Parts:TPS61299YBHR
- added JP1: SolderJumper_3_Bridged12, symbol Jumper:SolderJumper_3_Bridged12
- added L2: WIP252010P-1R0ML, easyeda2kicad:IND-SMD_L2.5-W2.0, symbol EasyEda2Kicad:WIP252010P-1R0ML
- added R24: 10k, easyeda2kicad:R0402, symbol Device:R
- added R25: 100k, symbol Device:R
- added R26, R27: 22, symbol Device:R
- added R28, R29: 10k, symbol Device:R
- added RN2: 100k, easyeda2kicad:RES-ARRAY-SMD_16P-L3.8-W1.6-P0.50-BL, symbol EasyEda2Kicad:R_Pack08_Split
- added SW1, SW2: TS-3025-B-C-B, easyeda2kicad:SW-SMD_L3.0-W2.5-P3.40-LS4.0-L, symbol EasyEda2Kicad:TS-3025-B-C-B
- added U11, U8: AGM60P90A, easyeda2kicad:TDSON-8_L5.9-W5.2-P1.27-BL, symbol EasyEda2Kicad:AGM60P90A
- added U12: SY6280AAAC, easyeda2kicad:TSOT-23-5_L2.9-W1.6-P0.95-LS2.8-BL, symbol EasyEda2Kicad:SY6280AAAC
- added U2: TS3A5223RSWR, easyeda2kicad:QFN-10_L1.4-W1.8-P0.40-BL, symbol EasyEda2Kicad:TS3A5223RSWR
- added U4: LM66200DRLR, easyeda2kicad:SOT-583-8_L2.1-W1.2-P0.50-LS1.6-BL, symbol EasyEda2Kicad:LM66200DRLR
- added U5: FSA2567UMX, easyeda2kicad:UMLP-16_L2.6-W1.8-P0.40-BL, symbol EasyEda2Kicad:FSA2567UMX
- added U6, U7: 74HC4051PW,118, easyeda2kicad:TSSOP-16_L5.0-W4.4-P0.65-LS6.4-BL, symbol EasyEda2Kicad:74HC4051PW,118
- added U9: 74AHC1G14SE-7, easyeda2kicad:SOT-353_L2.1-W1.3-P0.65-LS2.3-BR, symbol EasyEda2Kicad:74AHC1G14SE-7
- D1: now not fitted; now left out of the parts list
- R10, R11: value R -> 100k
- R9: renamed from R5; value R -> 100k
- gave numbers to parts that had none: 3
- renumbered C7 to C4, Cout3 to Cout1, Cout1 to Cout2, Cout2 to Cout3, D3 to D2, L2 to L1, R6 to R12, R17 to R13, R18 to R14, R20 to R15, R13 to R16, R14 to R17, R15 to R18, R16 to R19, R21 to R20, R22 to R21, R23 to R22, R24 to R23, R1 to R3, R2 to R4, R8 to R5, R9 to R6, R4 to R7, R3 to R8, U2 to U10, U6 to U3
Connections:
- net 3V3: now also R10.1, R11.1, R7.1, R8.1, R9.1, U3.5 (VDD), C3.2, JP1.3 (B), R28.1, R29.1, RN2.10 (R7.2), RN2.11 (R6.2), RN2.12 (R5.2), RN2.13 (R4.2), RN2.14 (R3.2), RN2.15 (R2.2), RN2.16 (R1.2), U4.2 (VOUT), U4.7 (VOUT), U5.14 (VCC), U6.16 (VCC), U7.16 (VCC), U9.5 (VCC); no longer C4.1, Cout2.2, Cout3.2, L1.1, Rpg1.2, Rtfb1.1
- net CC1: now also D3.1 (CH1)
- net CC2: now also D3.5 (CH4)
- net DN: now also D3.2 (CH2), R26.1
- net DP: now also D3.4 (CH3), R27.1
- net GND: now also U10.1 (IO45), U10.2 (IO48), C10.1, C11.2, C2.1, C3.1, C5.2, C6.2, C7.2, C8.2, C9.2 (-), D3.3 (GND_1), D3.8 (GND_2), IC3.A2 (GND), JP1.1 (A), R24.2, R25.2, SW1.1, SW2.1, U12.2 (GND), U4.1 (GND), U4.4 (~{ON}), U4.5 (GND), U5.6 (GND), U6.4 (Y7), U6.6 (~{E}), U6.7 (VEE), U6.8 (GND), U7.4 (Y7), U7.7 (VEE), U7.8 (GND), U9.3 (GND); no longer R10.1, R11.1, U3.12 (EN_N)
- net INT: now also R9.2; no longer R9.1
- net SCL: now also U5.13 (1DAT)
- net SDA: now also U5.5 (1RST)
- net at R20.1: now also U7.15 (Y2)
- net at U3.9 (SDA/SNK_VSET): now also U5.4 (RST)
- net at R17.1: now also U6.14 (Y1)
- net at R22.1: now also U7.13 (Y0)
- net at U3.10 (SCL/SNK_ISET): now also U5.12 (DAT)
- net at R12.2: now also U6.1 (Y4)
- net at R19.1: now also U6.12 (Y3)
- net at R18.1: now also U6.13 (Y0)
- net at R16.1: now also U6.15 (Y2)
- net pwrsrc_ind: now reaches R10.2
- net pwrsrc_ind: now also U4.8 (ST)
- net i2c_gpio_SEL: now reaches R11.2
- net i2c_gpio_SEL: now also U10.8 (IO7), U5.2 (Sel)
- net VbusOUT: now reaches Q1.1 (D)
- net at R13.2: now also U7.1 (Y4)
- net at R21.1: now also U7.14 (Y1)
- net at R4.1: now also U5.8 (CLK)
- net at R23.1: now also U7.12 (Y3)
- net at R15.2: now also U7.5 (Y5)
- net at R14.2: now also U7.2 (Y6)
- new net: RN2.2 (R2.1), U6.10 (S1)
- new net: RN2.1 (R1.1), U6.11 (S0)
- new net: U5.3 (2RST), U6.3 (Z)
- new net: RN2.3 (R3.1), U6.9 (S2)
- new net: IC3.C2 (VSEL), R25.1
- new net: C11.1, R29.2, SW1.2, U10.12 (IO36)
- new net: R24.1, U12.3 (ISET)
- new net: RN2.7 (R7.1), U9.2 (A)
- new net: R27.2, U10.1 (IO45)
- new net: R26.2, U10.2 (IO48)
- new net: RN2.6 (R6.1), U7.9 (S2)
- new net: JP1.2 (C), U5.9 (1CLK)
- new net: C6.1, C8.1, C9.1 (+), IC3.A1 (VIN), IC3.C1 (EN), L2.1, U12.1 (OUT)
- new net: IC3.B1 (SW), L2.2
- new net: U5.11 (2DAT), U7.3 (Z)
- new net: U7.6 (~{E}), U9.4 (Y)
- new net: RN2.4 (R4.1), U7.11 (S0)
- new net: RN2.5 (R5.1), U7.10 (S1)
- new net 3V2bck: C7.1, IC3.B2 (VOUT), U4.6 (VIN2)
- new net 3V3smps: C2.2, C4.1, C5.1, Cout2.2, Cout3.2, L1.1, Rpg1.2, Rtfb1.1, U12.4 (EN), U12.5 (IN), U4.3 (VIN1)
- new net EN: C10.2, R28.2, SW2.2, U10.12 (IO36)
- new net ENnPD: U3.12 (EN_N)
- no-connect marks 2 -> 15
Other:
- note added: "0k 1.25A 2k26 1.5A 4k02 1.75A 6k04 2A 8k45 2.25A 11k5 2.5A 15k8 2.75A 21k 3A NC(E=H)3.25A subst RDSon from ALL!"
- note added: "A variant without output discharge Iset=6800/R"
- note added: "HHH = A7 = GND = select 5V 0k 5V 3k 9V 6k04 12V 11k 15V 19k1 20V open 28V (20V) subst RDSon from ALL!"
- note added: "HUSB238A Open(2CLK) GPIO mode 2+3(VDD) I2C 62H 2+1(GND) I2C 42H"
- note removed: "Open GPIO mode 2+1(VDD) I2C 62H 2+3(GND) I2C 42H"
- moved on the sheet: C1, C4, Cboot1, Cin1, Cinx1, Cout1, Cout2, Cout3, Cvcc1, D2, IC1, L1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
